Commit message: V1.15

File: ranger_sim/ranger_mini_gazebo/xacro/livox_mid360.xacro (robot description, xacro)
@@ -6,12 +6,18 @@
   <xacro:property name="laser_max_range" value="200.0"/>
   <xacro:property name="ros_topic" value="scan"/>
-  <xacro:property name="samples" value="24000"/>
+  <!-- <xacro:property name="samples" value="24000"/> -->
+  <xacro:property name="samples" value="5000"/>
   <xacro:property name="downsample" value="1"/>
   <xacro:macro name="null_inertial">
-    <inertial>
+    <!-- <inertial>
       <mass value="0.1"/>
     <inertia ixx="0.01" ixy="0" ixz="0"
           iyy="0.01" iyz="0"
           izz="0.01"/>
+    </inertial> -->
+    <inertial>
+      <mass value="1e-5" />
+      <origin xyz="0 0 0" rpy="0 0 0"/>
+      <inertia ixx="1e-6" ixy="0" ixz="0" iyy="1e-6" iyz="0" izz="1e-6" />
     </inertial>
   </xacro:macro>
@@ -32,5 +38,5 @@
       </visual>
       <collision>
-		  <origin xyz="0 0 0" rpy="0 0 0" />
+		    <origin xyz="0 0 0" rpy="0 0 0" />
         <geometry>
           <mesh filename="package://ranger_mini_gazebo/description/meshes/livox_mid360/livox_mid360.dae" >
@@ -45,5 +51,5 @@
       <parent link="base"/>
       <child link="base_scan"/>
-      <origin rpy="0 0 0" xyz="0.0 1.0 0.2"/>
+      <origin rpy="0 0 0" xyz="0.0 0.0 0.2"/>
   </joint>
   <!--xacro:macro name="Livox_Mid_gazebo_sensor" params="visualize:=True
@@ -51,43 +57,44 @@
                   noise_stddev:=0.01 name:=livox"-->
   <gazebo reference="base_scan">
-      <sensor type="ray" name="livox_sensor">
+      <sensor type="ray" name="laser_livox">
         <pose>0 0 0 0 0 0</pose>
         <visualize>true</visualize>
-        <update_rate>10</update_rate>
+        <update_rate>40</update_rate>
         <!-- This ray plgin is only for visualization. -->
         <plugin name="gazebo_ros_laser_controller" filename="liblivox_laser_simulation.so">
-        <!-- <plugin name="gazebo_ros_head_hokuyo_controller" filename="libgazebo_ros_laser.so"> -->
-			<ray>
-			  <scan>
-				<horizontal>
-				<samples>100</samples>
-				<resolution>1</resolution>
-				<min_angle>${0}</min_angle>
-				<max_angle>${2*M_PI}</max_angle>
-				</horizontal>
-				<vertical>
-				<samples>360</samples>
-				<resolution>1</resolution>
-				<min_angle>${-7.22/180*M_PI}</min_angle>
-				<max_angle>${55.22/180*M_PI}</max_angle>
-				</vertical>
-			  </scan>
-			  <range>
-				<min>${laser_min_range}</min>
-				<max>${laser_max_range}</max>
-				<resolution>0.002</resolution>
-			  </range>
-			  <noise>
-				<type>gaussian</type>
-				<mean>0.0</mean>
-				<stddev>0.01</stddev>
-			  </noise>
-			</ray>
-          <visualize>true</visualize>
-		  <samples>${samples}</samples>
-		  <downsample>${downsample}</downsample>
-		  <csv_file_name>package://ranger_mini_gazebo/scan_mode/mid360.csv</csv_file_name>
-		  <ros_topic>${ros_topic}</ros_topic>
-      <frameName>base_scan</frameName>
+        <ray>
+			    <scan>
+				    <horizontal>
+				      <samples>100</samples>
+				      <resolution>1</resolution>
+				      <min_angle>${0}</min_angle>
+				      <max_angle>${2*M_PI}</max_angle>
+				    </horizontal>
+				    <vertical>
+				      <samples>360</samples>
+				      <resolution>1</resolution>
+				      <min_angle>${-7.22/180*M_PI}</min_angle>
+				      <max_angle>${55.22/180*M_PI}</max_angle>
+				    </vertical>
+			    </scan>
+			    <range>
+				    <min>${laser_min_range}</min>
+				    <max>${laser_max_range}</max>
+				    <resolution>0.002</resolution>
+			    </range>
+			    <noise>
+				    <type>gaussian</type>
+				    <mean>0.0</mean>
+				    <stddev>0.01</stddev>
+			    </noise>
+			  </ray>
+        <visualize>true</visualize>
+		    <samples>${samples}</samples>
+		    <downsample>${downsample}</downsample>
+		    <csv_file_name>package://ranger_mini_gazebo/scan_mode/mid360.csv</csv_file_name>
+		    <!-- <plugin name="gazebo_ros_laser_controller" filename="liblivox_laser_simulation.so"> -->
+        <ros_topic>${ros_topic}</ros_topic>
+          <!-- <topicName>/scan</topicName> -->
+        <!-- <frameName>base_scan</frameName> -->
         </plugin>
       </sensor>

Commit message: V1.15

File: ranger_sim/ranger_mini_gazebo/xacro/livox_mid360.xacro (robot description, xacro)
@@ -4,5 +4,5 @@
   <xacro:property name="M_PI" value="3.14159"/>
   <xacro:property name="laser_min_range" value="0.1"/>
-  <xacro:property name="laser_max_range" value="200.0"/>
+  <xacro:property name="laser_max_range" value="100.0"/>
   <xacro:property name="ros_topic" value="scan"/>
   <!-- <xacro:property name="samples" value="24000"/> -->
@@ -66,5 +66,5 @@
 			    <scan>
 				    <horizontal>
-				      <samples>100</samples>
+				      <samples>450</samples>
 				      <resolution>1</resolution>
 				      <min_angle>${0}</min_angle>
@@ -72,5 +72,5 @@
 				    </horizontal>
 				    <vertical>
-				      <samples>360</samples>
+				      <samples>100</samples>
 				      <resolution>1</resolution>
 				      <min_angle>${-7.22/180*M_PI}</min_angle>
